Commit message: Add joint to ros2 control

File: urdf/crane_x7.ros2_control.xacro (robot description, xacro)
@@ -122,4 +122,14 @@
         <param name="current_to_effort">2.20</param>
       </joint>
+      <joint name="${name_joint_gripper_finger_b}">
+        <command_interface name="position">
+          <param name="min">${joint_hand_lower_limit}</param>
+          <param name="max">${joint_hand_upper_limit}</param>
+        </command_interface>
+        <state_interface name="position"/>
+        <state_interface name="velocity"/>
+        <state_interface name="effort"/>
+        <param name="current_to_effort">2.20</param>
+      </joint>
     </ros2_control>
   </xacro:macro>
