Commit message: Port to Harmonic

File: urdf/crane_x7.gazebo.xacro (robot description, xacro)
@@ -49,5 +49,5 @@
             ">
     <gazebo>
-      <plugin filename="libign_ros2_control-system.so" name="ign_ros2_control::IgnitionROS2ControlPlugin">
+      <plugin filename="libgz_ros2_control-system.so" name="gz_ros2_control::GazeboSimROS2ControlPlugin">
         <parameters>$(find ${config_package})/${config_file_path}</parameters>
       </plugin>

File: urdf/crane_x7.gazebo_ros2_control.xacro (robot description, xacro)
@@ -11,4 +11,5 @@
             name_joint_7
             name_joint_gripper_finger_a
+            name_joint_gripper_finger_b
             joint_1_lower_limit
             joint_1_upper_limit
@@ -30,5 +31,5 @@
     <ros2_control name="${name}" type="system">
       <hardware>
-        <plugin>ign_ros2_control/IgnitionSystem</plugin>
+        <plugin>gz_ros2_control/GazeboSimSystem</plugin>
       </hardware>
       <joint name="${name_joint_1}">
@@ -104,4 +105,12 @@
         <state_interface name="effort"/>
       </joint>
+    <joint name="${name_joint_gripper_finger_b}">
+      <param name="mimic">${name_joint_gripper_finger_a}</param>
+      <param name="multiplier">1</param>
+      <command_interface name="position"/>
+      <state_interface name="position"/>
+      <state_interface name="velocity"/>
+      <state_interface name="effort"/>
+    </joint>
     </ros2_control>
   </xacro:macro>
