Commit message: Jazzy対応 (#10)
* Update README

* Update README.md

* gz_ros2_control対応

* authorに溝口追加

* CIのymlファイルをjazzyに対応

* READMEのJazzy対応

* gz_sim対応

* gitignore復元

* CIのコメント修正

* Update README

* コメント修正

* スタイル修正

* Update README

* mimic joint修正

* author更新

---------

Co-authored-by: ShotaAk <s.aoki@rt-net.jp>
Co-authored-by: mizonon <mizoguchi@rt-net.jp>

File: urdf/crane_x7.gazebo_ros2_control.xacro (robot description, xacro)
@@ -31,5 +31,5 @@
     <ros2_control name="${name}" type="system">
       <hardware>
-        <plugin>ign_ros2_control/IgnitionSystem</plugin>
+        <plugin>gz_ros2_control/GazeboSimSystem</plugin>
       </hardware>
       <joint name="${name_joint_1}">
@@ -105,12 +105,11 @@
         <state_interface name="effort"/>
       </joint>
-    <joint name="${name_joint_gripper_finger_b}">
-      <param name="mimic">${name_joint_gripper_finger_a}</param>
-      <param name="multiplier">1</param>
-      <command_interface name="position"/>
-      <state_interface name="position"/>
-      <state_interface name="velocity"/>
-      <state_interface name="effort"/>
-    </joint>
+      <joint name="${name_joint_gripper_finger_b}">
+        <param name="mimic">${name_joint_gripper_finger_a}</param>
+        <param name="multiplier">1</param>
+        <state_interface name="position"/>
+        <state_interface name="velocity"/>
+        <state_interface name="effort"/>
+      </joint>
     </ros2_control>
   </xacro:macro>
