Commit message: joint_4の可動範囲を調整 (#11)

File: urdf/crane_x7.urdf.xacro (robot description, xacro)
@@ -86,5 +86,5 @@
   <xacro:property name="JOINT_3_UPPER_LIMIT" value="${radians(157)}"/>
   <!-- JOINT_4はサーボ可動範囲を超えやすいため、LOWER_LIMITをサーボのリミット値より小さくする -->
-  <xacro:property name="JOINT_4_LOWER_LIMIT" value="${radians(-159)}"/>
+  <xacro:property name="JOINT_4_LOWER_LIMIT" value="${radians(-161)}"/>
   <!-- Gazeboの挙動がlimit付近で不安定なためUPPER_LIMITをサーボのリミット値より大きくする -->
   <!-- 参照: https://github.com/rt-net/crane_x7_ros/pull/162 -->

Commit message: joint2の可動範囲調整 (#13)

File: urdf/crane_x7.urdf.xacro (robot description, xacro)
@@ -82,6 +82,6 @@
   <xacro:property name="JOINT_1_LOWER_LIMIT" value="${radians(-157)}"/>
   <xacro:property name="JOINT_1_UPPER_LIMIT" value="${radians(157)}"/>
-  <xacro:property name="JOINT_2_LOWER_LIMIT" value="${radians(-90)}"/>
-  <xacro:property name="JOINT_2_UPPER_LIMIT" value="${radians(90)}"/>
+  <xacro:property name="JOINT_2_LOWER_LIMIT" value="${radians(-92)}"/>
+  <xacro:property name="JOINT_2_UPPER_LIMIT" value="${radians(92)}"/>
   <xacro:property name="JOINT_3_LOWER_LIMIT" value="${radians(-157)}"/>
   <xacro:property name="JOINT_3_UPPER_LIMIT" value="${radians(157)}"/>
